File: fuel_capacity_sensor.kicad_pcb (KiCad board)
At the start: 2 copper layers, 69 parts, among them J2 Conn_02x03_Counter_Clockwise, J3 Conn_01x01, J4 Conn_01x01, Q1 2N2222a, SW1 SW_Push, U1 LT1762EMS8-5, U2 LM324, U3 ADuM1201CR, U4 DCP01B, U5 LM324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

Commit message: Updated schematic and footprints
Parts:
- added D6: YLW, Diodes_SMD:D_SOD-123F, F.Cu at (137.8, 68.0)
- added J1: Conn_01x06_Male, Connectors_JST:JST_XH_B06B-XH-A_06x2.50mm_Straight, F.Cu at (104.2, 64.6)
- added J5: Conn_01x06_Male, Pin_Headers:Pin_Header_Straight_1x06_Pitch2.54mm, F.Cu at (208.8, 111.4)
- added R25: 1K, Resistors_SMD:R_0603, F.Cu at (136.8, 75.8)
- added TP1: TEST, Measurement_Points:Test_Point_Keystone_5015_Micro-Minature, F.Cu at (146.6, 76.2)
- added TP2: TEST, Measurement_Points:Test_Point_Keystone_5015_Micro-Minature, F.Cu at (147.2, 69.8)
- added TP3: TEST, Measurement_Points:Test_Point_Keystone_5015_Micro-Minature, F.Cu at (155.0, 85.4)
- added TP4: TEST, Measurement_Points:Test_Point_Keystone_5015_Micro-Minature, F.Cu at (161.8, 85.2)
- J2: value Conn_02x03_Counter_Clockwise -> Conn_01x06_Male; footprint Pin_Headers:Pin_Header_Straight_2x03_Pitch2.54mm -> Connectors_JST:JST_XH_B06B-XH-A_06x2.50mm_Straight
- J3: value Conn_01x01 -> Conn_02x03_Counter_Clockwise; footprint CustomComponents:FASTON-187-vert-90deg-terminal -> Pin_Headers:Pin_Header_Straight_2x03_Pitch2.54mm
- J4: value Conn_01x01 -> Conn_Coaxial; footprint CustomComponents:FASTON-187-vert-90deg-terminal -> Connectors:bnc-ci
- moved J4 86.6 mm to (81.0, 79.2)
- moved J2 72.5 mm to (104.6, 74.6)
- moved J3 33.2 mm to (162.0, 123.8)
Connections:
- C13 pad 2: GNDS -> CAN-GND
- C14 pad 2: GNDS -> CAN-GND
- J2 pad 1: PDO -> CAN-SHLD
- J2 pad 2: SCK -> +12V
- J2 pad 3: RESET -> CAN-GND
- J2 pad 4: GND -> CAN-HI
- J2 pad 5: PDI -> CAN-LO
- J2 pad 6: Net-(J2-Pad6) -> GND
- J3 pad 1: CAP-PLATE-1 -> PDO
- U3 pad 5: GNDS -> CAN-GND
- U4 pad 5: GNDS -> CAN-GND
- U6 pad 2: GNDS -> CAN-GND
- U6 pad 8: GNDS -> CAN-GND

Commit message: Many updates
Parts:
- added C24: 100nF, Capacitors_SMD:C_0603, F.Cu at (129.3, 79.4)
- added C25: 10nF, Capacitors_SMD:C_0603, F.Cu at (100.4, 111.8)
- added C26: 10nF, Capacitors_SMD:C_0603, F.Cu at (133.2, 108.7)
- added F1: Fuse, Fuse_Holders_and_Fuses:Fuse_SMD1206_Reflow, F.Cu at (99.7, 83.1)
- added REF**: MountingHole_2.7mm, Mounting_Holes:MountingHole_2.7mm, F.Cu at (157.0, 117.0)
- added REF**: MountingHole_2.7mm, Mounting_Holes:MountingHole_2.7mm, F.Cu at (157.0, 73.0)
- added REF**: MountingHole_2.7mm, Mounting_Holes:MountingHole_2.7mm, F.Cu at (93.0, 117.0)
- added REF**: MountingHole_2.7mm, Mounting_Holes:MountingHole_2.7mm, F.Cu at (100.0, 87.5)
- added TP5: TEST, Measurement_Points:Test_Point_Keystone_5015_Micro-Minature, F.Cu at (124.9, 118.4)
- added TP6: TEST, Measurement_Points:Test_Point_Keystone_5015_Micro-Minature, F.Cu at (130.1, 118.4)
- C2: value 1uF -> .33uF
- C5: value 10nF -> 100nF
- C6: value 10uF -> 100nF
- J1: value Conn_01x06_Male -> CAN1
- J2: value Conn_01x06_Male -> CAN2
- J3: value Conn_02x03_Counter_Clockwise -> ISP
- J5: value Conn_01x06_Male -> SERIAL
- Q1: value 2N2222a -> BCW65CLT1G; footprint TO_SOT_Packages_THT:TO-92_Inline_Narrow_Oval -> TO_SOT_Packages_SMD:SOT-23
- U1: value LT1762EMS8-5 -> LM78M05_TO252; footprint Housings_SSOP:MSOP-8_3x3mm_Pitch0.65mm -> TO_SOT_Packages_SMD:TO-252-2
- U2: value LM324 -> LT1491A; footprint Housings_SOIC:SOIC-16W_5.3x10.2mm_Pitch1.27mm -> Housings_SOIC:SOIC-16_3.9x9.9mm_Pitch1.27mm
- U5: value LM324 -> LT1490A; footprint Housings_SOIC:SOIC-16W_5.3x10.2mm_Pitch1.27mm -> Housings_SOIC:SOIC-8_3.9x4.9mm_Pitch1.27mm
- moved C17 95.3 mm to (128.4, 92.3), turned to 180 degrees
- moved SW1 94.6 mm to (131.6, 96.3)
- moved R24 92.8 mm to (131.7, 92.3), turned to 180 degrees
- moved D2 91.5 mm to (148.8, 72.6), turned to 90 degrees
- moved C5 85.7 mm to (139.1, 79.0), turned to 270 degrees
- moved R13 85.3 mm to (148.9, 77.1)
- moved RV3 77.4 mm to (122.1, 93.9)
- moved RV2 74.7 mm to (112.8, 93.9)
- moved RV1 74.0 mm to (103.5, 93.9)
- moved TP2 68.5 mm to (92.6, 111.1)
- moved C2 68.1 mm to (140.9, 104.7)
- moved U2 67.6 mm to (107.6, 111.4)
- moved TP4 65.4 mm to (105.5, 118.4), turned to 180 degrees
- moved TP3 64.0 mm to (100.2, 118.4)
- moved D5 62.9 mm to (145.6, 72.6), turned to 90 degrees
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Connections:
- C5 pad 1: VDD -> GND
- C5 pad 2: Net-(C5-Pad2) -> VDD
- J1 pad 2: +12V -> Net-(F1-Pad2)
- J2 pad 2: +12V -> Net-(F1-Pad2)
- J5 pad 2: Net-(J5-Pad2) -> GND
- Q1 pad 2: Net-(Q1-Pad2) -> VCC
- Q1 pad 3: VCC -> Net-(Q1-Pad3)
- R2 pad 1: Net-(Q1-Pad2) -> Net-(Q1-Pad3)
- TP2 pad 1: Net-(R11-Pad1) -> CAP-PLATE-2
- U1 pad 1: VDD -> +12V
- U1 pad 2: VDD -> GND
- U1 pad 3: Net-(C5-Pad2) -> VDD
- U5 pad 4: VCC -> CAP-PLATE-2
- U5 pad 8: (no net) -> VCC
Other:
- board outline added: 70 x 50 mm

Commit message: Fixed ISP header
Connections:
- J3 pad 2: SCK -> Net-(J3-Pad2)
- J3 pad 3: RESET -> SCK
- J3 pad 4: GND -> PDI
- J3 pad 5: PDI -> RESET
- J3 pad 6: Net-(J3-Pad6) -> GND
Changed lines of the file:
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@@
     (links 178)
     (no_connects 174)
-    (area 84.871429 68.325 165.128572 123.275)
+    (area 89.924999 69.924999 160.075001 120.075001)
     (thickness 1.6)
     (drawings 6)
@@
   (net 100 "Net-(D6-Pad2)")
   (net 101 CAN-SHLD)
-  (net 102 "Net-(J3-Pad6)")
-  (net 103 "Net-(J5-Pad3)")
-  (net 104 "Net-(J5-Pad6)")
-  (net 105 "Net-(F1-Pad2)")
-  (net 106 "Net-(Q1-Pad3)")
+  (net 102 "Net-(J5-Pad3)")
+  (net 103 "Net-(J5-Pad6)")
+  (net 104 "Net-(F1-Pad2)")
+  (net 105 "Net-(Q1-Pad3)")
+  (net 106 "Net-(J3-Pad2)")
   (net_class Default "This is the default net class."
     (clearance 0.2)
@@
     (add_net "Net-(D6-Pad2)")
     (add_net "Net-(F1-Pad2)")
-    (add_net "Net-(J3-Pad6)")
+    (add_net "Net-(J3-Pad2)")
     (add_net "Net-(J5-Pad3)")
     (add_net "Net-(J5-Pad6)")
@@
     (fp_line (start 1.25 0.7) (end -1.25 0.7) (layer F.CrtYd) (width 0.05))
     (pad 1 smd rect (at -0.75 0 180) (size 0.5 0.9) (layers F.Cu F.Paste F.Mask)
-      (net 106 "Net-(Q1-Pad3)"))
+      (net 105 "Net-(Q1-Pad3)"))
     (pad 2 smd rect (at 0.75 0 180) (size 0.5 0.9) (layers F.Cu F.Paste F.Mask)
       (net 27 +12V))
@@
       (net 101 CAN-SHLD))
     (pad 2 thru_hole circle (at 2.5 0) (size 1.75 1.75) (drill 1) (layers *.Cu *.Mask)
-      (net 105 "Net-(F1-Pad2)"))
+      (net 104 "Net-(F1-Pad2)"))
     (pad 3 thru_hole circle (at 5 0) (size 1.75 1.75) (drill 1) (layers *.Cu *.Mask)
       (net 98 CAN-GND))
@@
       (net 25 PDO))
     (pad 2 thru_hole oval (at 2.54 0) (size 1.7 1.7) (drill 1) (layers *.Cu *.Mask)
-      (net 24 SCK))
+      (net 106 "Net-(J3-Pad2)"))
     (pad 3 thru_hole oval (at 0 2.54) (size 1.7 1.7) (drill 1) (layers *.Cu *.Mask)
-      (net 17 RESET))
+      (net 24 SCK))
     (pad 4 thru_hole oval (at 2.54 2.54) (size 1.7 1.7) (drill 1) (layers *.Cu *.Mask)
-      (net 3 GND))
-    (pad 5 thru_hole oval (at 0 5.08) (size 1.7 1.7) (drill 1) (layers *.Cu *.Mask)
       (net 26 PDI))
+    (pad 5 thru_hole oval (at 0 5.08) (size 1.7 1.7) (drill 1) (layers *.Cu *.Mask)
+      (net 17 RESET))
     (pad 6 thru_hole oval (at 2.54 5.08) (size 1.7 1.7) (drill 1) (layers *.Cu *.Mask)
-      (net 102 "Net-(J3-Pad6)"))
+      (net 3 GND))
     (model ${KISYS3DMOD}/Pin_Headers.3dshapes/Pin_Header_Straight_2x03_Pitch2.54mm.wrl
       (at (xyz 0 0 0))
@@
       (net 101 CAN-SHLD))
     (pad 2 thru_hole circle (at 2.5 0) (size 1.75 1.75) (drill 1) (layers *.Cu *.Mask)
-      (net 105 "Net-(F1-Pad2)"))
+      (net 104 "Net-(F1-Pad2)"))
     (pad 3 thru_hole circle (at 5 0) (size 1.75 1.75) (drill 1) (layers *.Cu *.Mask)
       (net 98 CAN-GND))
@@
       (net 3 GND))
     (pad 3 thru_hole oval (at 0 5.08) (size 1.7 1.7) (drill 1) (layers *.Cu *.Mask)
-      (net 103 "Net-(J5-Pad3)"))
+      (net 102 "Net-(J5-Pad3)"))
     (pad 4 thru_hole oval (at 0 7.62) (size 1.7 1.7) (drill 1) (layers *.Cu *.Mask)
       (net 61 RX))
@@
       (net 62 TX))
     (pad 6 thru_hole oval (at 0 12.7) (size 1.7 1.7) (drill 1) (layers *.Cu *.Mask)
-      (net 104 "Net-(J5-Pad6)"))
+      (net 103 "Net-(J5-Pad6)"))
     (model ${KISYS3DMOD}/Pin_Headers.3dshapes/Pin_Header_Straight_1x06_Pitch2.54mm.wrl
       (at (xyz 0 0 0))
@@
       (net 27 +12V))
     (pad 2 smd rect (at 1.2 0 90) (size 2.03 1.14) (layers F.Cu F.Paste F.Mask)
-      (net 105 "Net-(F1-Pad2)"))
+      (net 104 "Net-(F1-Pad2)"))
   )
   (module Mounting_Holes:MountingHole_2.7mm (layer F.Cu)
@@
       (net 2 VCC))
     (pad 3 smd rect (at 1 0) (size 0.9 0.8) (layers F.Cu F.Paste F.Mask)
-      (net 106 "Net-(Q1-Pad3)"))
+      (net 105 "Net-(Q1-Pad3)"))
     (model ${KISYS3DMOD}/TO_SOT_Packages_SMD.3dshapes/SOT-23.wrl
       (at (xyz 0 0 0))

Commit message: New version of kicad changes
Parts:
- U7: value AT90CAN32-16AU -> AT90CAN64-16AU
- moved REF** 16.1 mm to (93.0, 73.0)
- moved C5 14.3 mm to (135.8, 92.9)
- moved C24 13.8 mm to (126.6, 92.9)
- moved U3 11.3 mm to (131.1, 91.6)
- moved SW1 7.10 mm to (131.8, 103.4)
- moved C17 7.01 mm to (128.7, 99.3)
- moved R24 7.00 mm to (131.8, 99.3)
- moved U6 5.66 mm to (130.9, 82.1)
- moved C14 5.63 mm to (131.0, 86.9)
- moved J4 5.60 mm to (101.8, 76.0)
- moved C13 5.12 mm to (121.6, 91.4)
- moved U4 5.08 mm to (117.7, 84.4)
- moved C8 5.04 mm to (111.4, 91.4)
- moved J1 4.50 mm to (110.7, 73.3)
- moved J2 4.30 mm to (129.4, 73.3)
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Changed lines of the file:
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@@
     (47 F.CrtYd user)
     (48 B.Fab user)
-    (49 F.Fab user)
+    (49 F.Fab user hide)
   )
   (setup
@@
   )
   (module Capacitors_SMD:C_0603 (layer F.Cu)
-    (at 106.5 90.2)
+    (at 111.4 91.4)
     (descr "Capacitor SMD 0603, reflow soldering, AVX (see smccp.pdf)")
     (tags "capacitor 0603")
@@
   )
   (module Capacitors_SMD:C_0603 (layer F.Cu)
-    (at 116.6 90.3 180)
+    (at 121.6 91.4 180)
     (descr "Capacitor SMD 0603, reflow soldering, AVX (see smccp.pdf)")
     (tags "capacitor 0603")
@@
   )
   (module Capacitors_SMD:C_0603 (layer F.Cu)
-    (at 126.3 90 180)
+    (at 131 86.9 180)
     (descr "Capacitor SMD 0603, reflow soldering, AVX (see smccp.pdf)")
     (tags "capacitor 0603")
@@
   )
   (module Capacitors_SMD:C_0603 (layer F.Cu)
-    (at 128.4 92.3 180)
+    (at 128.7 99.3 180)
     (descr "Capacitor SMD 0603, reflow soldering, AVX (see smccp.pdf)")
     (tags "capacitor 0603")
@@
   )
   (module Diodes_SMD:D_SOD-123F (layer F.Cu)
-    (at 148.8 72.6 90)
+    (at 152 72.6 90)
     (descr D_SOD-123F)
     (tags D_SOD-123F)
@@
   )
   (module Diodes_SMD:D_SOD-123F (layer F.Cu)
-    (at 145.6 72.6 90)
+    (at 149.2 72.6 90)
     (descr D_SOD-123F)
     (tags D_SOD-123F)
@@
   )
   (module Resistors_SMD:R_0603 (layer F.Cu)
-    (at 148.9 77.1)
+    (at 152.1 77.1)
     (descr "Resistor SMD 0603, reflow soldering, Vishay (see dcrcw.pdf)")
     (tags "resistor 0603")
@@
   )
   (module Resistors_SMD:R_0603 (layer F.Cu)
-    (at 145.6 77.1)
+    (at 149.3 77.1)
     (descr "Resistor SMD 0603, reflow soldering, Vishay (see dcrcw.pdf)")
     (tags "resistor 0603")
@@
   )
   (module Resistors_SMD:R_0603 (layer F.Cu)
-    (at 131.7 92.3 180)
+    (at 131.8 99.3 180)
     (descr "Resistor SMD 0603, reflow soldering, Vishay (see dcrcw.pdf)")
     (tags "resistor 0603")
@@
   )
   (module Housings_SOIC:SOIC-8_3.9x4.9mm_Pitch1.27mm (layer F.Cu)
-    (at 133.9 80.7 180)
+    (at 131.1 91.6 180)
     (descr "8-Lead Plastic Small Outline (SN) - Narrow, 3.90 mm Body [SOIC] (see Microchip Packaging Specification 00000049BS.pdf)")
     (tags "SOIC 1.27")
@@
       (effects (font (size 1 1) (thickness 0.15)))
     )
-    (fp_text value ADuM1201CR (at 0 3.5 180) (layer F.Fab)
+    (fp_text value ADuM1201CR (at 0 3.5 180) (layer F.Fab) hide
       (effects (font (size 1 1) (thickness 0.15)))
     )
@@
   )
   (module Housings_SOIC:SOIC-8_3.9x4.9mm_Pitch1.27mm (layer F.Cu)
-    (at 126.3 85.4 90)
+    (at 130.9 82.1 90)
     (descr "8-Lead Plastic Small Outline (SN) - Narrow, 3.90 mm Body [SOIC] (see Microchip Packaging Specification 00000049BS.pdf)")
     (tags "SOIC 1.27")
@@
       (effects (font (size 1 1) (thickness 0.15)))
     )
-    (fp_text value MCP2551-I/SN (at 0 3.5 90) (layer F.Fab)
+    (fp_text value MCP2551-I/SN (at 0 3.5 90) (layer F.Fab) hide
       (effects (font (size 1 1) (thickness 0.15)))
     )
@@
       (effects (font (size 1 1) (thickness 0.15)))
     )
-    (fp_text value AT90CAN32-16AU (at 0 7.45 90) (layer F.Fab)
+    (fp_text value AT90CAN64-16AU (at 0 7.45 90) (layer F.Fab) hide
       (effects (font (size 1 1) (thickness 0.15)))
     )
@@
   )
   (module CustomComponents:switch-kpt-1187B-SMD (layer F.Cu)
-    (at 131.6 96.3)
+    (at 131.8 103.4)
     (tags switch)
     (fp_text reference SW1 (at -0.3 3.9) (layer F.SilkS)
@@
   )
   (module CustomComponents:DCP01B_SO_7_14 (layer F.Cu)
-    (at 112.7 83.5 90)
+    (at 117.7 84.4 90)
     (fp_text reference U4 (at -0.1016 1.016 90) (layer F.SilkS)
       (effects (font (size 1.016 0.762) (thickness 0.127)))
@@
   )
   (module Diodes_SMD:D_SOD-123F (layer F.Cu)
-    (at 142.4 72.6 90)
+    (at 146.4 72.6 90)
     (descr D_SOD-123F)
     (tags D_SOD-123F)
@@
   )
   (module Connectors_JST:JST_XH_B06B-XH-A_06x2.50mm_Straight (layer F.Cu)
-    (at 106.2 73.4)
+    (at 110.7 73.3)
     (descr "JST XH series connector, B06B-XH-A, top entry type, through hole")
     (tags "connector jst xh tht top vertical 2.50mm")
@@
   )
   (module Connectors:bnc-ci (layer F.Cu)
-    (at 96.2 76.2)
+    (at 101.8 76)
     (descr "BNC female PCB mount 4 pin straight chassis connector")
     (tags "BNC female PCB mount 4 pin straight chassis connector http://img-asia.electrocomponents.com/largeimages/L457024-02.gif")
@@
       (effects (font (size 1 1) (thickness 0.15)))
     )
-    (fp_text value Conn_Coaxial (at 0 6.5) (layer F.Fab)
+    (fp_text value Conn_Coaxial (at 0 6.5) (layer F.Fab) hide
       (effects (font (size 1 1) (thickness 0.15)))
     )
@@
   )
   (module Resistors_SMD:R_0603 (layer F.Cu)
-    (at 142.3 77.1)
+    (at 146.6 77.1)
     (descr "Resistor SMD 0603, reflow soldering, Vishay (see dcrcw.pdf)")
     (tags "resistor 0603")
@@
   )
   (module Connectors_JST:JST_XH_B06B-XH-A_06x2.50mm_Straight (layer F.Cu)
-    (at 125.1 73.4)
+    (at 129.4 73.3)
     (descr "JST XH series connector, B06B-XH-A, top entry type, through hole")
     (tags "connector jst xh tht top vertical 2.50mm")
@@
       (effects (font (size 1 1) (thickness 0.15)))
     )
-    (fp_text value SERIAL (at 0 15.03) (layer F.Fab)
+    (fp_text value SERIAL (at 0 15.03) (layer F.Fab) hide
       (effects (font (size 1 1) (thickness 0.15)))
     )
@@
       (effects (font (size 1 1) (thickness 0.15)))
     )
-    (fp_text value LM78M05_TO252 (at 0 4.5) (layer F.Fab)
+    (fp_text value LM78M05_TO252 (at 0 4.5) (layer F.Fab) hide
       (effects (font (size 1 1) (thickness 0.15)))
     )
@@
   )
   (module Fuse_Holders_and_Fuses:Fuse_SMD1206_Reflow (layer F.Cu)
-    (at 99.7 83.1)
+    (at 99.9 84.1)
     (descr "Fuse, Sicherung, SMD1206, Littlefuse-Wickmann, Reflow,")
     (tags "Fuse Sicherung SMD1206 Littlefuse-Wickmann Reflow ")
@@
     (tags "mounting hole 2.7mm no annular")
     (attr virtual)
-    (fp_text reference REF** (at 0 -3.7) (layer F.SilkS)
+    (fp_text reference REF** (at 0 -3.7) (layer F.SilkS) hide
       (effects (font (size 1 1) (thickness 0.15)))
     )
-    (fp_text value MountingHole_2.7mm (at 0 3.7) (layer F.Fab)
+    (fp_text value MountingHole_2.7mm (at 0 3.7) (layer F.Fab) hide
       (effects (font (size 1 1) (thickness 0.15)))
     )
@@
     (tags "mounting hole 2.7mm no annular")
     (attr virtual)
-    (fp_text reference REF** (at 0 -3.7) (layer F.SilkS)
+    (fp_text reference REF** (at 0 -3.7) (layer F.SilkS) hide
       (effects (font (size 1 1) (thickness 0.15)))
     )
-    (fp_text value MountingHole_2.7mm (at 0 3.7) (layer F.Fab)
+    (fp_text value MountingHole_2.7mm (at 0 3.7) (layer F.Fab) hide
       (effects (font (size 1 1) (thickness 0.15)))
     )
@@
     (tags "mounting hole 2.7mm no annular")
     (attr virtual)
-    (fp_text reference REF** (at -1.1 5.2) (layer F.SilkS)
+    (fp_text reference REF** (at -1.1 5.2) (layer F.SilkS) hide
       (effects (font (size 1 1) (thickness 0.15)))
     )
-    (fp_text value MountingHole_2.7mm (at 0 3.7) (layer F.Fab)
+    (fp_text value MountingHole_2.7mm (at 0 3.7) (layer F.Fab) hide
       (effects (font (size 1 1) (thickness 0.15)))
     )
@@
   )
   (module Mounting_Holes:MountingHole_2.7mm (layer F.Cu)
-    (at 100 87.5)
+    (at 93 73)
     (descr "Mounting Hole 2.7mm, no annular")
     (tags "mounting hole 2.7mm no annular")
     (attr virtual)
-    (fp_text reference REF** (at 0 -3.7) (layer F.SilkS)
+    (fp_text reference REF** (at 0 -3.7) (layer F.SilkS) hide
       (effects (font (size 1 1) (thickness 0.15)))
     )
-    (fp_text value MountingHole_2.7mm (at 0 3.7) (layer F.Fab)
+    (fp_text value MountingHole_2.7mm (at 0 3.7) (layer F.Fab) hide
       (effects (font (size 1 1) (thickness 0.15)))
     )
@@
       (effects (font (size 1 1) (thickness 0.15)))
     )
-    (fp_text value BCW65CLT1G (at 0 2.5) (layer F.Fab)
+    (fp_text value BCW65CLT1G (at 0 2.5) (layer F.Fab) hide
       (effects (font (size 1 1) (thickness 0.15)))
     )
@@
   )
   (module Capacitors_SMD:C_0603 (layer F.Cu)
-    (at 139.1 79 270)
+    (at 135.8 92.9 270)
     (descr "Capacitor SMD 0603, reflow soldering, AVX (see smccp.pdf)")
     (tags "capacitor 0603")
@@
   )
   (module Capacitors_SMD:C_0603 (layer F.Cu)
-    (at 129.3 79.4 270)
+    (at 126.6 92.9 270)
     (descr "Capacitor SMD 0603, reflow soldering, AVX (see smccp.pdf)")
     (tags "capacitor 0603")
